Commit message: Add files via upload

File: robot_proyecto_description/urdf/robot_proyecto.xacro (robot description, xacro)
@@ -4,4 +4,9 @@
 <xacro:include filename="$(find robot_proyecto_description)/urdf/robot_proyecto.trans" />
 <xacro:include filename="$(find robot_proyecto_description)/urdf/robot_proyecto.gazebo" />
+<link name="world" />
+<joint name="world_to_base_link=" type="fixed">
+     <parent link="world"/>
+     <child link="base_link"/>
+</joint>
 <link name="base_link">
   <inertial>
@@ -13,5 +18,5 @@
     <origin xyz="0 0 0" rpy="0 0 0"/>
     <geometry>
-      <mesh filename="package://robot_proyecto_description/meshes/base_link.stl" scale="0.001 0.001 0.001"/>
+      <mesh filename="package://robot_proyecto_description/meshes/base_link.stl" />
     </geometry>
     <material name="silver"/>
@@ -20,5 +25,5 @@
     <origin xyz="0 0 0" rpy="0 0 0"/>
     <geometry>
-      <mesh filename="package://robot_proyecto_description/meshes/base_link.stl" scale="0.001 0.001 0.001"/>
+      <mesh filename="package://robot_proyecto_description/meshes/base_link.stl" />
     </geometry>
   </collision>
@@ -33,5 +38,5 @@
     <origin xyz="0.0 -0.0 -0.116" rpy="0 0 0"/>
     <geometry>
-      <mesh filename="package://robot_proyecto_description/meshes/link2_1.stl" scale="0.001 0.001 0.001"/>
+      <mesh filename="package://robot_proyecto_description/meshes/link2_1.stl"/>
     </geometry>
     <material name="silver"/>
@@ -40,5 +45,5 @@
     <origin xyz="0.0 -0.0 -0.116" rpy="0 0 0"/>
     <geometry>
-      <mesh filename="package://robot_proyecto_description/meshes/link2_1.stl" scale="0.001 0.001 0.001"/>
+      <mesh filename="package://robot_proyecto_description/meshes/link2_1.stl"/>
     </geometry>
   </collision>
@@ -53,5 +58,5 @@
     <origin xyz="-0.0 0.005 -0.311" rpy="0 0 0"/>
     <geometry>
-      <mesh filename="package://robot_proyecto_description/meshes/link3_1.stl" scale="0.001 0.001 0.001"/>
+      <mesh filename="package://robot_proyecto_description/meshes/link3_1.stl"/>
     </geometry>
     <material name="silver"/>
@@ -60,5 +65,5 @@
     <origin xyz="-0.0 0.005 -0.311" rpy="0 0 0"/>
     <geometry>
-      <mesh filename="package://robot_proyecto_description/meshes/link3_1.stl" scale="0.001 0.001 0.001"/>
+      <mesh filename="package://robot_proyecto_description/meshes/link3_1.stl"/>
     </geometry>
   </collision>
@@ -73,5 +78,5 @@
     <origin xyz="-0.0 -0.025 -0.338" rpy="0 0 0"/>
     <geometry>
-      <mesh filename="package://robot_proyecto_description/meshes/link4_1.stl" scale="0.001 0.001 0.001"/>
+      <mesh filename="package://robot_proyecto_description/meshes/link4_1.stl"/>
     </geometry>
     <material name="silver"/>
@@ -80,5 +85,5 @@
     <origin xyz="-0.0 -0.025 -0.338" rpy="0 0 0"/>
     <geometry>
-      <mesh filename="package://robot_proyecto_description/meshes/link4_1.stl" scale="0.001 0.001 0.001"/>
+      <mesh filename="package://robot_proyecto_description/meshes/link4_1.stl"/>
     </geometry>
   </collision>
@@ -93,5 +98,5 @@
     <origin xyz="-0.0 -0.203 -0.337766" rpy="0 0 0"/>
     <geometry>
-      <mesh filename="package://robot_proyecto_description/meshes/link5_1.stl" scale="0.001 0.001 0.001"/>
+      <mesh filename="package://robot_proyecto_description/meshes/link5_1.stl"/>
     </geometry>
     <material name="silver"/>
@@ -100,5 +105,5 @@
     <origin xyz="-0.0 -0.203 -0.337766" rpy="0 0 0"/>
     <geometry>
-      <mesh filename="package://robot_proyecto_description/meshes/link5_1.stl" scale="0.001 0.001 0.001"/>
+      <mesh filename="package://robot_proyecto_description/meshes/link5_1.stl"/>
     </geometry>
   </collision>
@@ -113,5 +118,5 @@
     <origin xyz="-0.0 -0.228 -0.338" rpy="0 0 0"/>
     <geometry>
-      <mesh filename="package://robot_proyecto_description/meshes/link6_1.stl" scale="0.001 0.001 0.001"/>
+      <mesh filename="package://robot_proyecto_description/meshes/link6_1.stl"/>
     </geometry>
     <material name="silver"/>
@@ -120,5 +125,5 @@
     <origin xyz="-0.0 -0.228 -0.338" rpy="0 0 0"/>
     <geometry>
-      <mesh filename="package://robot_proyecto_description/meshes/link6_1.stl" scale="0.001 0.001 0.001"/>
+      <mesh filename="package://robot_proyecto_description/meshes/link6_1.stl"/>
     </geometry>
   </collision>
@@ -133,5 +138,5 @@
     <origin xyz="-0.0 -0.0 -0.05" rpy="0 0 0"/>
     <geometry>
-      <mesh filename="package://robot_proyecto_description/meshes/link1_1.stl" scale="0.001 0.001 0.001"/>
+      <mesh filename="package://robot_proyecto_description/meshes/link1_1.stl"/>
     </geometry>
     <material name="silver"/>
@@ -140,5 +145,5 @@
     <origin xyz="-0.0 -0.0 -0.05" rpy="0 0 0"/>
     <geometry>
-      <mesh filename="package://robot_proyecto_description/meshes/link1_1.stl" scale="0.001 0.001 0.001"/>
+      <mesh filename="package://robot_proyecto_description/meshes/link1_1.stl"/>
     </geometry>
   </collision>
